Commit message: met

File: src/articubot_one/description/robot_core.xacro (robot description, xacro)
@@ -10,5 +10,5 @@
     <xacro:property name="wheel_mass" value="0.05"/>
     <xacro:property name="wheel_offset_x" value="0.07"/>
-    <xacro:property name="wheel_offset_y" value="0.094"/>
+    <xacro:property name="wheel_offset_y" value="0.0925"/>
     <xacro:property name="wheel_offset_z" value="0.025"/>
     <xacro:property name="caster_wheel_radius" value="0.03"/>

File: src/articubot_one/description/ros2_control.xacro (robot description, xacro)
@@ -8,5 +8,5 @@
                 <param name="left_wheel_name">left_wheel_joint</param>
                 <param name="right_wheel_name">right_wheel_joint</param>
-                <param name="loop_rate">30</param>
+                <param name="loop_rate">50</param>
                 <param name="device">/dev/ttyACM0</param>
                 <param name="baud_rate">57600</param>
