Commit message: nckh

File: src/articubot_one/description/lidar.xacro (robot description, xacro)
@@ -2,7 +2,6 @@
 <robot xmlns:xacro="http://www.ros.org/wiki/xacro" >
     <joint name="laser_joint" type="fixed">
-        <parent link="chassis"/>
-        <child link="laser_frame"/>
-        <origin xyz="0.135 0 0.1075" rpy="0 0 0"/>
+        <parent link="base_link"/>  <child link="laser_frame"/>
+        <origin xyz="0.08 0 0.1425" rpy="0 0 0"/>
     </joint>
     <link name="laser_frame">

File: src/articubot_one/description/robot_core.xacro (robot description, xacro)
@@ -3,6 +3,6 @@
     <xacro:include filename="inertial_macros.xacro"/>
     <xacro:property name="chassis_length" value="0.3"/>
-    <xacro:property name="chassis_width" value="0.19"/>
-    <xacro:property name="chassis_height" value="0.09"/>
+    <xacro:property name="chassis_width" value="0.21"/>
+    <xacro:property name="chassis_height" value="0.10"/>
     <xacro:property name="chassis_mass" value="1.5"/>
     <xacro:property name="wheel_radius" value="0.0325"/>
@@ -10,10 +10,10 @@
     <xacro:property name="wheel_mass" value="0.05"/>
     <xacro:property name="wheel_offset_x" value="0.07"/>
-    <xacro:property name="wheel_offset_y" value="0.11"/>
-    <xacro:property name="wheel_offset_z" value="0.01"/>
-    <xacro:property name="caster_wheel_radius" value="0.01"/>
+    <xacro:property name="wheel_offset_y" value="0.094"/>
+    <xacro:property name="wheel_offset_z" value="0.025"/>
+    <xacro:property name="caster_wheel_radius" value="0.03"/>
     <xacro:property name="caster_wheel_mass" value="0.01"/>
-    <xacro:property name="caster_wheel_offset_x" value="0.22"/>
-    <xacro:property name="caster_wheel_offset_z" value="${wheel_offset_z - wheel_radius + caster_wheel_radius}"/>
+    <xacro:property name="caster_wheel_offset_x" value="0.176"/>
+    <xacro:property name="caster_wheel_offset_z" value="${-wheel_radius + caster_wheel_radius}"/>
     <material name="white">
         <color rgba="1 1 1 1" />
@@ -46,5 +46,5 @@
         <parent link="base_link"/>
         <child link="chassis"/>
-        <origin xyz="${-wheel_offset_x} 0 ${-wheel_offset_z}"/>
+        <origin xyz="${-wheel_offset_x} 0 ${wheel_offset_z}" rpy="0 0 0"/>
     </joint>
     <link name="chassis">
@@ -123,7 +123,7 @@
     <!-- CASTER WHEEL LINK -->
     <joint name="caster_wheel_joint" type="fixed">
-        <parent link="chassis"/>
+        <parent link="base_link"/>
         <child link="caster_wheel"/>
-        <origin xyz="${caster_wheel_offset_x} 0 ${caster_wheel_offset_z}"/>
+        <origin xyz="${caster_wheel_offset_x} 0 ${caster_wheel_offset_z}" rpy="0 0 0"/>
     </joint>
     <link name="caster_wheel">

Commit message: cuc

File: src/articubot_one/description/lidar.xacro (robot description, xacro)
@@ -12,11 +12,4 @@
             <material name="black"/>
         </visual>
-        <!-- <visual>
-            <origin xyz="0 0 -0.05"/>
-            <geometry>
-                <cylinder radius="0.01" length="0.1"/>
-            </geometry>
-            <material name="black"/>
-        </visual> -->
         <collision>
             <geometry>

File: src/articubot_one/description/robot_core.xacro (robot description, xacro)
@@ -31,14 +31,14 @@
         <color rgba="1 0 0 1"/>
     </material>
+    <!-- BASE_FOOTPRINT LINK (ROOT) -->
+    <link name="base_footprint">
+    </link>
     <!-- BASE LINK -->
+    <joint name="base_footprint_joint" type="fixed">
+        <parent link="base_footprint"/>
+        <child link="base_link"/>
+        <origin xyz="0 0 ${wheel_radius}" rpy="0 0 0"/>
+    </joint>
     <link name="base_link">
-    </link>
-    <!-- BASE_FOOTPRINT LINK -->
-    <joint name="base_footprint_joint" type="fixed">
-        <parent link="base_link"/>
-        <child link="base_footprint"/>
-        <origin xyz="0 0 0" rpy="0 0 0"/>
-    </joint>
-    <link name="base_footprint">
     </link>
     <!-- CHASSIS LINK -->

File: src/articubot_one/description/ros2_control.xacro (robot description, xacro)
@@ -1,5 +1,6 @@
 <?xml version="1.0"?>
 <robot xmlns:xacro="http://www.ros.org/wiki/xacro">
-    <xacro:unless value="${sim_mode == 'true'}">
+    <xacro:arg name="sim_mode" default="false"/>
+    <xacro:unless value="$(arg sim_mode)">
         <ros2_control name="RealRobot" type="system">
             <hardware>
@@ -31,5 +32,5 @@
         </ros2_control>
     </xacro:unless>
-    <xacro:if value="${sim_mode == 'true'}">
+    <xacro:if value="$(arg sim_mode)">
         <ros2_control name="GazeboSystem" type="system">
             <hardware>
@@ -53,10 +54,10 @@
             </joint>
         </ros2_control>
+        <gazebo>
+            <plugin name="gazebo_ros2_control" filename="libgazebo_ros2_control.so">
+                <parameters>$(find articubot_one)/config/my_controllers.yaml</parameters>
+                <parameters>$(find articubot_one)/config/gaz_ros2_ctl_use_sim.yaml</parameters>
+            </plugin>
+        </gazebo>
     </xacro:if>
-    <gazebo>
-        <plugin name="gazebo_ros2_control" filename="libgazebo_ros2_control.so">
-            <parameters>$(find articubot_one)/config/my_controllers.yaml</parameters>
-            <parameters>$(find articubot_one)/config/gaz_ros2_ctl_use_sim.yaml</parameters>
-        </plugin>
-    </gazebo>
 </robot>

Commit message: new

File: src/articubot_one/description/lidar.xacro (robot description, xacro)
@@ -12,4 +12,11 @@
             <material name="black"/>
         </visual>
+        <!-- <visual>
+            <origin xyz="0 0 -0.05"/>
+            <geometry>
+                <cylinder radius="0.01" length="0.1"/>
+            </geometry>
+            <material name="black"/>
+        </visual> -->
         <collision>
             <geometry>

File: src/articubot_one/description/robot_core.xacro (robot description, xacro)
@@ -10,5 +10,5 @@
     <xacro:property name="wheel_mass" value="0.05"/>
     <xacro:property name="wheel_offset_x" value="0.07"/>
-    <xacro:property name="wheel_offset_y" value="0.0925"/>
+    <xacro:property name="wheel_offset_y" value="0.094"/>
     <xacro:property name="wheel_offset_z" value="0.025"/>
     <xacro:property name="caster_wheel_radius" value="0.03"/>
@@ -31,14 +31,14 @@
         <color rgba="1 0 0 1"/>
     </material>
-    <!-- BASE_FOOTPRINT LINK (ROOT) -->
+    <!-- BASE LINK -->
+    <link name="base_link">
+    </link>
+    <!-- BASE_FOOTPRINT LINK -->
+    <joint name="base_footprint_joint" type="fixed">
+        <parent link="base_link"/>
+        <child link="base_footprint"/>
+        <origin xyz="0 0 0" rpy="0 0 0"/>
+    </joint>
     <link name="base_footprint">
-    </link>
-    <!-- BASE LINK -->
-    <joint name="base_footprint_joint" type="fixed">
-        <parent link="base_footprint"/>
-        <child link="base_link"/>
-        <origin xyz="0 0 ${wheel_radius}" rpy="0 0 0"/>
-    </joint>
-    <link name="base_link">
     </link>
     <!-- CHASSIS LINK -->

File: src/articubot_one/description/ros2_control.xacro (robot description, xacro)
@@ -1,6 +1,5 @@
 <?xml version="1.0"?>
 <robot xmlns:xacro="http://www.ros.org/wiki/xacro">
-    <xacro:arg name="sim_mode" default="false"/>
-    <xacro:unless value="$(arg sim_mode)">
+    <xacro:unless value="${'$(arg sim_mode)' == 'true'}">
         <ros2_control name="RealRobot" type="system">
             <hardware>
@@ -8,5 +7,5 @@
                 <param name="left_wheel_name">left_wheel_joint</param>
                 <param name="right_wheel_name">right_wheel_joint</param>
-                <param name="loop_rate">50</param>
+                <param name="loop_rate">30</param>
                 <param name="device">/dev/ttyACM0</param>
                 <param name="baud_rate">57600</param>
@@ -32,5 +31,5 @@
         </ros2_control>
     </xacro:unless>
-    <xacro:if value="$(arg sim_mode)">
+    <xacro:if value="${'$(arg sim_mode)' == 'true'}">
         <ros2_control name="GazeboSystem" type="system">
             <hardware>
@@ -54,10 +53,10 @@
             </joint>
         </ros2_control>
-        <gazebo>
-            <plugin name="gazebo_ros2_control" filename="libgazebo_ros2_control.so">
-                <parameters>$(find articubot_one)/config/my_controllers.yaml</parameters>
-                <parameters>$(find articubot_one)/config/gaz_ros2_ctl_use_sim.yaml</parameters>
-            </plugin>
-        </gazebo>
     </xacro:if>
+    <gazebo>
+        <plugin name="gazebo_ros2_control" filename="libgazebo_ros2_control.so">
+            <parameters>$(find articubot_one)/config/my_controllers.yaml</parameters>
+            <parameters>$(find articubot_one)/config/gaz_ros2_ctl_use_sim.yaml</parameters>
+        </plugin>
+    </gazebo>
 </robot>
